File: Drawing/Final project.kicad_sch (KiCad schematic)
At the start: 7 parts, among them SW1 RotaryEncoder_Switch, SW2 SW_Push_Open, U1 MOUDLE-SEEEDUINO-XIAO-ESP32C3, U2 module_adxl345

Commit message: Add files via upload
Parts:
- added J1: SpeakON_NL2, symbol Connector_Audio:SpeakON_NL2
- added M1: Fan, symbol Motor:Fan
Connections:
- net GND: now also J1.1-, M1.2 (-)
- net at U1.1 (PA02_A0_D0): now also SW1.S1
- net at U1.10 (PA5_A9_D9_MISO): now also SW1.A; no longer SW1.S1
- net at U1.11 (PA6_A10_D10_MOSI): now also J1.1+; no longer D1.3 (PAD)
- net at Brd1.2 (VCC), D1.2 (A), U1.12 (3V3)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: now also SW1.C, M1.1 (+)
- net at U1.2 (PA4_A1_D1): now also D1.3 (PAD)
- net at U1.9 (PA7_A8_D8_SCK): now also SW1.B
Other:
- moved on the sheet: D1, SW1
